Commit message: Fix Nav2 launc

File: puzzlebot_ws/src/puzzlebot_ros2/puzzlebot_description/urdf/puzzlebot.urdf.xacro (robot description, xacro)
@@ -1,196 +1,18 @@
 <?xml version="1.0"?>
-<robot name="puzzlebot">
-  <!-- ================= BASE FOOTPRINT ================= -->
-  <link name="base_footprint"/>
-  <!-- ================= BASE LINK ================= -->
-  <link name="base_link">
-    <visual>
-      <origin xyz="-0.052 0 0" rpy="0 0 0"/>
-      <geometry>
-        <mesh filename="package://puzzlebot_description/meshes/Puzzlebot_Jetson_Lidar_Edition_Base(1).stl" scale="1 1 1"/>
-      </geometry>
-      <material name="white">
-        <color rgba="1.0 1.0 1.0 1.0"/>
-      </material>
-    </visual>
-    <collision>
-      <origin xyz="-0.052 0 0.05" rpy="0 0 0"/>
-      <geometry>
-        <box size="0.20 0.14 0.10"/>
-      </geometry>
-    </collision>
-    <inertial>
-      <origin xyz="0 0 0"/>
-      <mass value="2.0"/>
-      <inertia ixx="0.01" ixy="0.0" ixz="0.0"
-               iyy="0.01" iyz="0.0"
-               izz="0.02"/>
-    </inertial>
-  </link>
-  <joint name="base_link_joint" type="fixed">
-    <parent link="base_footprint"/>
-    <child link="base_link"/>
-    <origin xyz="0.052 0 0.05" rpy="0 0 0"/>
-  </joint>
-  <!-- ================= LEFT WHEEL ================= -->
-  <link name="wheel_l_link">
-    <visual>
-      <origin xyz="0 0 0" rpy="1.5708 0 0"/>
-      <geometry>
-        <mesh filename="package://puzzlebot_description/meshes/Puzzlebot_Wheel.stl" scale="1 1 1"/>
-      </geometry>
-      <material name="gray">
-        <color rgba="0.2 0.2 0.2 1.0"/>
-      </material>
-    </visual>
-    <collision>
-      <origin xyz="0 0 0" rpy="1.5708 0 0"/>
-      <geometry>
-        <cylinder radius="0.0325" length="0.02"/>
-      </geometry>
-    </collision>
-    <inertial>
-      <mass value="0.2"/>
-      <inertia ixx="0.0002" ixy="0.0" ixz="0.0"
-               iyy="0.0002" iyz="0.0"
-               izz="0.0002"/>
-    </inertial>
-  </link>
-  <joint name="wheel_l_joint" type="continuous">
-    <parent link="base_link"/>
-    <child link="wheel_l_link"/>
-    <origin xyz="0.00 0.095 0.0" rpy="0 0 0"/>
-    <axis xyz="0 1 0"/>
-  </joint>
-  <!-- ================= RIGHT WHEEL ================= -->
-  <link name="wheel_r_link">
-    <visual>
-      <origin xyz="0 0 0" rpy="1.5708 0 0"/>
-      <geometry>
-        <mesh filename="package://puzzlebot_description/meshes/Puzzlebot_Wheel.stl" scale="1 1 1"/>
-      </geometry>
-      <material name="gray">
-        <color rgba="0.2 0.2 0.2 1.0"/>
-      </material>
-    </visual>
-    <collision>
-      <origin xyz="0 0 0" rpy="1.5708 0 0"/>
-      <geometry>
-        <cylinder radius="0.0325" length="0.02"/>
-      </geometry>
-    </collision>
-    <inertial>
-      <mass value="0.2"/>
-      <inertia ixx="0.0002" ixy="0.0" ixz="0.0"
-               iyy="0.0002" iyz="0.0"
-               izz="0.0002"/>
-    </inertial>
-  </link>
-  <joint name="wheel_r_joint" type="continuous">
-    <parent link="base_link"/>
-    <child link="wheel_r_link"/>
-    <origin xyz="0.00 -0.095 0.0" rpy="0 0 0"/>
-    <axis xyz="0 1 0"/>
-  </joint>
-  <!-- ================= CASTER WHEEL ================= -->
-  <link name="caster_link">
-    <visual>
-      <origin xyz="0 0 0" rpy="0 0 0"/>
-      <geometry>
-        <mesh filename="package://puzzlebot_description/meshes/Puzzlebot_Caster_Wheel.stl" scale="1 1 1"/>
-      </geometry>
-      <material name="black">
-        <color rgba="0.0 0.0 0.0 1.0"/>
-      </material>
-    </visual>
-    <collision>
-      <origin xyz="0 0 0" rpy="0 0 0"/>
-      <geometry>
-        <sphere radius="0.015"/>
-      </geometry>
-    </collision>
-    <inertial>
-      <mass value="0.05"/>
-      <inertia ixx="0.00001" ixy="0.0" ixz="0.0"
-               iyy="0.00001" iyz="0.0"
-               izz="0.00001"/>
-    </inertial>
-  </link>
-  <joint name="caster_joint" type="fixed">
-    <parent link="base_link"/>
-    <child link="caster_link"/>
-    <origin xyz="-0.147 0 -0.045" rpy="0 0 0"/>
-  </joint>
-  <!-- ================= LIDAR ================= -->
-  <link name="lidar_link">
-    <visual>
-      <origin xyz="0 0 0" rpy="0 0 0"/>
-      <geometry>
-        <cylinder radius="0.035" length="0.05"/>
-      </geometry>
-      <material name="red">
-        <color rgba="1 0 0 1"/>
-      </material>
-    </visual>
-    <collision>
-      <origin xyz="0 0 0" rpy="0 0 0"/>
-      <geometry>
-        <cylinder radius="0.035" length="0.05"/>
-      </geometry>
-    </collision>
-    <inertial>
-      <mass value="0.1"/>
-      <inertia ixx="0.0001" ixy="0.0" ixz="0.0"
-               iyy="0.0001" iyz="0.0"
-               izz="0.0001"/>
-    </inertial>
-  </link>
-  <joint name="lidar_joint" type="fixed">
-    <parent link="base_link"/>
-    <child link="lidar_link"/>
-    <origin xyz="0.00 0 0.10" rpy="0 0 0"/>
-  </joint>
-  <!-- ================= GAZEBO LIDAR ================= -->
-  <gazebo reference="lidar_link">
-    <sensor name="lidar" type="gpu_lidar">
-      <always_on>true</always_on>
-      <visualize>true</visualize>
-      <update_rate>20</update_rate>
-      <topic>/scan</topic>
-      <frame_id>lidar_link</frame_id>
-      <ray>
-        <scan>
-          <horizontal>
-            <samples>360</samples>
-            <resolution>1</resolution>
-            <min_angle>-3.14159</min_angle>
-            <max_angle>3.14159</max_angle>
-          </horizontal>
-        </scan>
-        <range>
-          <min>0.05</min>
-          <max>10.0</max>
-          <resolution>0.01</resolution>
-        </range>
-      </ray>
-    </sensor>
-  </gazebo>
-  <!-- ================= GAZEBO PLUGINS ================= -->
-  <gazebo>
-    <plugin filename="ignition-gazebo-joint-state-publisher-system"
-            name="ignition::gazebo::systems::JointStatePublisher"/>
-    <plugin filename="ignition-gazebo-diff-drive-system"
-            name="ignition::gazebo::systems::DiffDrive">
-      <left_joint>wheel_l_joint</left_joint>
-      <right_joint>wheel_r_joint</right_joint>
-      <wheel_separation>0.19</wheel_separation>
-      <wheel_radius>0.0325</wheel_radius>
-      <topic>/cmd_vel</topic>
-      <odom_topic>/odom</odom_topic>
-      <tf_topic>/diff_drive/tf</tf_topic>
-      <frame_id>odom</frame_id>
-      <child_frame_id>base_footprint</child_frame_id>
-      <odom_publish_frequency>60</odom_publish_frequency>
-    </plugin>
-  </gazebo>
+<robot xmlns:xacro="http://www.ros.org/wiki/xacro" name="puzzlebot">
+  <xacro:arg name="prefix" default="" />
+  <xacro:include filename="$(find puzzlebot_description)/urdf/puzzlebot_base.urdf.xacro"/>
+  <xacro:include filename="$(find puzzlebot_description)/urdf/puzzlebot_control.xacro"/>
+  <xacro:include filename="$(find puzzlebot_description)/urdf/rpi_lidar_sensor.xacro"/>
+  <xacro:puzzlebot_base prefix="$(arg prefix)"/>
+  <xacro:rpi_lidar_sensor
+    prefix="$(arg prefix)"
+    frame_name="lidar_link"
+    parent="base_link"
+    topic_name="scan"
+    update_rate="20"
+    min_range="0.05"
+    max_range="10.0"
+    visualize="true"/>
+  <xacro:puzzlebot_control prefix="$(arg prefix)"/>
 </robot>

File: puzzlebot_ws/src/puzzlebot_ros2/puzzlebot_description/urdf/puzzlebot.xacro (robot description, xacro)
@@ -1,6 +1,8 @@
-<!-- ================= entry point ================= -->
 <?xml version="1.0"?>
 <robot xmlns:xacro="https://www.ros.org/wiki/xacro" name="puzzlebot">
+    <!-- ================= entry point ================= -->
+    <xacro:arg name="prefix" default="" />
     <xacro:include filename="$(find puzzlebot_description)/urdf/puzzlebot_base.urdf.xacro"/>
     <xacro:include filename="$(find puzzlebot_description)/urdf/puzzlebot_control.xacro"/>
-<robot>
+    <xacro:puzzlebot_control prefix="$(arg prefix)"/>
+</robot>

File: puzzlebot_ws/src/puzzlebot_ros2/puzzlebot_description/urdf/puzzlebot_base.urdf.xacro (robot description, xacro)
@@ -1,4 +1,176 @@
-<!-- ================= links y joints ================= -->
 <?xml version="1.0"?>
-<robot xmlns:xacro="https://www.ros.org/wiki/xacro" name="puzzlebot">
-<robot>
+<robot xmlns:xacro="http://www.ros.org/wiki/xacro">
+  <!-- estructura física del Puzzlebot   -->
+  <xacro:macro name="puzzlebot_base" params="prefix">
+    <!-- BASE FOOTPRINT                                           -->
+    <!-- Frame base del robot usado para navegación y TF         -->
+    <!-- Normalmente se coloca en el suelo, justo debajo del robot -->
+    <!-- ========================================================= -->
+    <link name="${prefix}base_footprint"/>
+    <!-- ========================================================= -->
+    <!-- BASE LINK                                                -->
+    <!-- Cuerpo principal del robot                              -->
+    <!-- Contiene mesh visual, colisión e inercia                -->
+    <!-- ========================================================= -->
+    <link name="${prefix}base_link">
+      <!-- ================= VISUAL ================= -->
+      <!-- Cómo se ve el robot en RViz/Gazebo -->
+      <visual>
+        <origin xyz="-0.052 0 0" rpy="0 0 0"/>
+        <geometry>
+          <mesh filename="package://puzzlebot_description/meshes/Puzzlebot_Jetson_Lidar_Edition_Base(1).stl"
+                scale="1 1 1"/>
+        </geometry>
+        <material name="white">
+          <color rgba="1.0 1.0 1.0 1.0"/>
+        </material>
+      </visual>
+      <!-- ================= COLLISION ================= -->
+      <!-- Geometría usada por Gazebo para física -->
+      <collision>
+        <origin xyz="-0.052 0 0.05" rpy="0 0 0"/>
+        <geometry>
+          <box size="0.20 0.14 0.10"/>
+        </geometry>
+      </collision>
+      <!-- ================= INERTIA ================= -->
+      <!-- Propiedades físicas del robot -->
+      <inertial>
+        <origin xyz="0 0 0"/>
+        <mass value="2.0"/>
+        <inertia
+          ixx="0.01" ixy="0.0" ixz="0.0"
+          iyy="0.01" iyz="0.0"
+          izz="0.02"/>
+      </inertial>
+    </link>
+    <!-- ========================================================= -->
+    <!-- JOINT BASE FOOTPRINT -> BASE LINK                        -->
+    <!-- Une el frame del suelo con el cuerpo del robot          -->
+    <!-- ========================================================= -->
+    <joint name="${prefix}base_link_joint" type="fixed">
+      <parent link="${prefix}base_footprint"/>
+      <child link="${prefix}base_link"/>
+      <origin xyz="0.052 0 0.05" rpy="0 0 0"/>
+    </joint>
+    <!-- ========================================================= -->
+    <!-- LLANTA IZQUIERDA                                         -->
+    <!-- ========================================================= -->
+    <link name="${prefix}wheel_l_link">
+      <!-- Visual -->
+      <visual>
+        <origin xyz="0 0 0" rpy="1.5708 0 0"/>
+        <geometry>
+          <mesh filename="package://puzzlebot_description/meshes/Puzzlebot_Wheel.stl"
+                scale="1 1 1"/>
+        </geometry>
+        <material name="gray">
+          <color rgba="0.2 0.2 0.2 1.0"/>
+        </material>
+      </visual>
+      <!-- Collision -->
+      <collision>
+        <origin xyz="0 0 0" rpy="1.5708 0 0"/>
+        <geometry>
+          <cylinder radius="0.0325" length="0.02"/>
+        </geometry>
+      </collision>
+      <!-- Inercia -->
+      <inertial>
+        <mass value="0.2"/>
+        <inertia
+          ixx="0.0002" ixy="0.0" ixz="0.0"
+          iyy="0.0002" iyz="0.0"
+          izz="0.0002"/>
+      </inertial>
+    </link>
+    <!-- Joint rueda izquierda -->
+    <joint name="${prefix}wheel_l_joint" type="continuous">
+      <parent link="${prefix}base_link"/>
+      <child link="${prefix}wheel_l_link"/>
+      <!-- Posición lateral izquierda -->
+      <origin xyz="0.00 0.095 0.0" rpy="0 0 0"/>
+      <!-- Eje de rotación -->
+      <axis xyz="0 1 0"/>
+    </joint>
+    <!-- ========================================================= -->
+    <!-- LLANTA DERECHA                                           -->
+    <!-- ========================================================= -->
+    <link name="${prefix}wheel_r_link">
+      <!-- Visual -->
+      <visual>
+        <origin xyz="0 0 0" rpy="1.5708 0 0"/>
+        <geometry>
+          <mesh filename="package://puzzlebot_description/meshes/Puzzlebot_Wheel.stl"
+                scale="1 1 1"/>
+        </geometry>
+        <material name="gray">
+          <color rgba="0.2 0.2 0.2 1.0"/>
+        </material>
+      </visual>
+      <!-- Collision -->
+      <collision>
+        <origin xyz="0 0 0" rpy="1.5708 0 0"/>
+        <geometry>
+          <cylinder radius="0.0325" length="0.02"/>
+        </geometry>
+      </collision>
+      <!-- Inercia -->
+      <inertial>
+        <mass value="0.2"/>
+        <inertia
+          ixx="0.0002" ixy="0.0" ixz="0.0"
+          iyy="0.0002" iyz="0.0"
+          izz="0.0002"/>
+      </inertial>
+    </link>
+    <!-- Joint rueda derecha -->
+    <joint name="${prefix}wheel_r_joint" type="continuous">
+      <parent link="${prefix}base_link"/>
+      <child link="${prefix}wheel_r_link"/>
+      <!-- Posición lateral derecha -->
+      <origin xyz="0.00 -0.095 0.0" rpy="0 0 0"/>
+      <!-- Eje de rotación -->
+      <axis xyz="0 1 0"/>
+    </joint>
+    <!-- ========================================================= -->
+    <!-- RUEDA CASTER                                              -->
+    <!-- Rueda loca trasera                                       -->
+    <!-- ========================================================= -->
+    <link name="${prefix}caster_link">
+      <!-- Visual -->
+      <visual>
+        <origin xyz="0 0 0" rpy="0 0 0"/>
+        <geometry>
+          <mesh filename="package://puzzlebot_description/meshes/Puzzlebot_Caster_Wheel.stl"
+                scale="1 1 1"/>
+        </geometry>
+        <material name="black">
+          <color rgba="0.0 0.0 0.0 1.0"/>
+        </material>
+      </visual>
+      <!-- Collision -->
+      <collision>
+        <origin xyz="0 0 0" rpy="0 0 0"/>
+        <geometry>
+          <sphere radius="0.015"/>
+        </geometry>
+      </collision>
+      <!-- Inercia -->
+      <inertial>
+        <mass value="0.05"/>
+        <inertia
+          ixx="0.00001" ixy="0.0" ixz="0.0"
+          iyy="0.00001" iyz="0.0"
+          izz="0.00001"/>
+      </inertial>
+    </link>
+    <!-- Joint caster -->
+    <joint name="${prefix}caster_joint" type="fixed">
+      <parent link="${prefix}base_link"/>
+      <child link="${prefix}caster_link"/>
+      <!-- Posición trasera -->
+      <origin xyz="-0.147 0 -0.045" rpy="0 0 0"/>
+    </joint>
+  </xacro:macro>
+</robot>

File: puzzlebot_ws/src/puzzlebot_ros2/puzzlebot_description/urdf/puzzlebot_control.xacro (robot description, xacro)
@@ -1,15 +1,15 @@
-<!-- ================= controller ================= -->
 <?xml version="1.0"?>
 <robot xmlns:xacro="https://www.ros.org/wiki/xacro">
+    <!-- ================= controller ================= -->
     <xacro:macro name="puzzlebot_control" params="prefix">
         <gazebo>
-            <plugin filename="gz-sim-sensores-system"
+            <plugin filename="gz-sim-sensors-system"
             name="gz::sim::systems::Sensors">
                 <render_engine>ogre2</render_engine>
             </plugin>
-            <plugin filename="gz-sim-dif-drive-system"
-            name="gz::sim::systems::DiffDRive">
-                <left_joint>${prefix}wheel_left_joint</left_joint>
-                <right_joint>${prefix}wheel_right_joint</right_joint>
+            <plugin filename="gz-sim-diff-drive-system"
+            name="gz::sim::systems::DiffDrive">
+                <left_joint>${prefix}wheel_l_joint</left_joint>
+                <right_joint>${prefix}wheel_r_joint</right_joint>
                 <wheel_separation>0.19</wheel_separation>
                 <wheel_radius>0.05</wheel_radius>
@@ -27,6 +27,6 @@
                 <topic>${prefix}joint_states</topic>
                 <update_rate>50</update_rate>
-                <joint_name>${prefix}wheel_left_joint</joint_name>
-                <joint_name>${prefix}wheel_right_joint</joint_name>
+                <joint_name>${prefix}wheel_l_joint</joint_name>
+                <joint_name>${prefix}wheel_r_joint</joint_name>
             </plugin>
         </gazebo>
