Commit message: Add code packages structure draft

File: puzzlebot_ws/src/puzzlebot_ros2/puzzlebot_description/urdf/puzzlebot.xacro (robot description, xacro)
@@ -3,6 +3,21 @@
     <!-- ================= entry point ================= -->
     <xacro:arg name="prefix" default="" />
+    <!-- Includes -->
     <xacro:include filename="$(find puzzlebot_description)/urdf/puzzlebot_base.urdf.xacro"/>
     <xacro:include filename="$(find puzzlebot_description)/urdf/puzzlebot_control.xacro"/>
+    <xacro:include filename="$(find puzzlebot_description)/urdf/rpi_lidar_sensor.xacro"/>
+    <!-- Robot base -->
+    <xacro:puzzlebot_base prefix="$(arg prefix)"/>
+    <!-- Lidar -->
+    <xacro:rpi_lidar_sensor
+        prefix="$(arg prefix)"
+        frame_name="lidar_link"
+        parent="base_link"
+        topic_name="scan"
+        update_rate="20"
+        min_range="0.05"
+        max_range="10.0"
+        visualize="true"/>
+    <!-- Gazebo control plugins -->
     <xacro:puzzlebot_control prefix="$(arg prefix)"/>
 </robot>

File: puzzlebot_ws/src/puzzlebot_ros2/puzzlebot_description/urdf/puzzlebot_base.urdf.xacro (robot description, xacro)
@@ -29,7 +29,7 @@
       <!-- Geometría usada por Gazebo para física -->
       <collision>
-        <origin xyz="-0.052 0 0.05" rpy="0 0 0"/>
+        <origin xyz="-0.052 0 0.015" rpy="0 0 0"/>
         <geometry>
-          <box size="0.20 0.14 0.10"/>
+          <box size="0.18 0.14 0.03"/>
         </geometry>
       </collision>
@@ -52,5 +52,5 @@
       <parent link="${prefix}base_footprint"/>
       <child link="${prefix}base_link"/>
-      <origin xyz="0.052 0 0.05" rpy="0 0 0"/>
+      <origin xyz="0.052 0 0.0325" rpy="0 0 0"/>
     </joint>
     <!-- ========================================================= -->
@@ -171,5 +171,5 @@
       <child link="${prefix}caster_link"/>
       <!-- Posición trasera -->
-      <origin xyz="-0.147 0 -0.045" rpy="0 0 0"/>
+      <origin xyz="-0.147 0 -0.0325" rpy="0 0 0"/>
     </joint>
   </xacro:macro>

File: puzzlebot_ws/src/puzzlebot_ros2/puzzlebot_description/urdf/puzzlebot_control.xacro (robot description, xacro)
@@ -13,5 +13,5 @@
                 <right_joint>${prefix}wheel_r_joint</right_joint>
                 <wheel_separation>0.19</wheel_separation>
-                <wheel_radius>0.05</wheel_radius>
+                <wheel_radius>0.0325</wheel_radius>
                 <topic>${prefix}cmd_vel</topic>
                 <tf_topic>${prefix}diff_drive/tf</tf_topic>

Commit message: Fixed robot position on Gazebo

File: puzzlebot_ws/src/puzzlebot_ros2/puzzlebot_description/urdf/puzzlebot.xacro (robot description, xacro)
@@ -3,21 +3,6 @@
     <!-- ================= entry point ================= -->
     <xacro:arg name="prefix" default="" />
-    <!-- Includes -->
     <xacro:include filename="$(find puzzlebot_description)/urdf/puzzlebot_base.urdf.xacro"/>
     <xacro:include filename="$(find puzzlebot_description)/urdf/puzzlebot_control.xacro"/>
-    <xacro:include filename="$(find puzzlebot_description)/urdf/rpi_lidar_sensor.xacro"/>
-    <!-- Robot base -->
-    <xacro:puzzlebot_base prefix="$(arg prefix)"/>
-    <!-- Lidar -->
-    <xacro:rpi_lidar_sensor
-        prefix="$(arg prefix)"
-        frame_name="lidar_link"
-        parent="base_link"
-        topic_name="scan"
-        update_rate="20"
-        min_range="0.05"
-        max_range="10.0"
-        visualize="true"/>
-    <!-- Gazebo control plugins -->
     <xacro:puzzlebot_control prefix="$(arg prefix)"/>
 </robot>

File: puzzlebot_ws/src/puzzlebot_ros2/puzzlebot_description/urdf/puzzlebot_base.urdf.xacro (robot description, xacro)
@@ -1,19 +1,9 @@
 <?xml version="1.0"?>
 <robot xmlns:xacro="http://www.ros.org/wiki/xacro">
-  <!-- estructura física del Puzzlebot   -->
   <xacro:macro name="puzzlebot_base" params="prefix">
-    <!-- BASE FOOTPRINT                                           -->
-    <!-- Frame base del robot usado para navegación y TF         -->
-    <!-- Normalmente se coloca en el suelo, justo debajo del robot -->
-    <!-- ========================================================= -->
     <link name="${prefix}base_footprint"/>
-    <!-- ========================================================= -->
-    <!-- BASE LINK                                                -->
-    <!-- Cuerpo principal del robot                              -->
-    <!-- Contiene mesh visual, colisión e inercia                -->
-    <!-- ========================================================= -->
+    <!-- ================= BASE LINK ================= -->
     <link name="${prefix}base_link">
-      <!-- ================= VISUAL ================= -->
-      <!-- Cómo se ve el robot en RViz/Gazebo -->
+      <!-- Visual -->
       <visual>
         <origin xyz="-0.052 0 0" rpy="0 0 0"/>
@@ -26,37 +16,29 @@
         </material>
       </visual>
-      <!-- ================= COLLISION ================= -->
-      <!-- Geometría usada por Gazebo para física -->
+      <!-- Collision -->
       <collision>
-        <origin xyz="-0.052 0 0.015" rpy="0 0 0"/>
+        <origin xyz="-0.052 0 0.05" rpy="0 0 0"/>
         <geometry>
-          <box size="0.18 0.14 0.03"/>
+          <box size="0.20 0.14 0.10"/>
         </geometry>
       </collision>
-      <!-- ================= INERTIA ================= -->
-      <!-- Propiedades físicas del robot -->
+      <!-- Inercia corregida -->
       <inertial>
-        <origin xyz="0 0 0"/>
-        <mass value="2.0"/>
+        <origin xyz="-0.02 0 -0.02"/>
+        <mass value="3.5"/>
         <inertia
-          ixx="0.01" ixy="0.0" ixz="0.0"
-          iyy="0.01" iyz="0.0"
-          izz="0.02"/>
+          ixx="0.06" ixy="0.0" ixz="0.0"
+          iyy="0.08" iyz="0.0"
+          izz="0.10"/>
       </inertial>
     </link>
-    <!-- ========================================================= -->
-    <!-- JOINT BASE FOOTPRINT -> BASE LINK                        -->
-    <!-- Une el frame del suelo con el cuerpo del robot          -->
-    <!-- ========================================================= -->
+    <!-- Joint base -->
     <joint name="${prefix}base_link_joint" type="fixed">
       <parent link="${prefix}base_footprint"/>
       <child link="${prefix}base_link"/>
-      <origin xyz="0.052 0 0.0325" rpy="0 0 0"/>
+      <origin xyz="0.052 0 0.07" rpy="0 0 0"/>
     </joint>
-    <!-- ========================================================= -->
-    <!-- LLANTA IZQUIERDA                                         -->
-    <!-- ========================================================= -->
+    <!-- ================= LEFT WHEEL ================= -->
     <link name="${prefix}wheel_l_link">
-      <!-- Visual -->
       <visual>
         <origin xyz="0 0 0" rpy="1.5708 0 0"/>
@@ -69,12 +51,10 @@
         </material>
       </visual>
-      <!-- Collision -->
       <collision>
         <origin xyz="0 0 0" rpy="1.5708 0 0"/>
         <geometry>
-          <cylinder radius="0.0325" length="0.02"/>
+          <cylinder radius="0.05" length="0.02"/>
         </geometry>
       </collision>
-      <!-- Inercia -->
       <inertial>
         <mass value="0.2"/>
@@ -85,18 +65,17 @@
       </inertial>
     </link>
-    <!-- Joint rueda izquierda -->
+    <!-- Fricción -->
+    <gazebo reference="${prefix}wheel_l_link">
+      <mu1>10.0</mu1>
+      <mu2>10.0</mu2>
+    </gazebo>
     <joint name="${prefix}wheel_l_joint" type="continuous">
       <parent link="${prefix}base_link"/>
       <child link="${prefix}wheel_l_link"/>
-      <!-- Posición lateral izquierda -->
       <origin xyz="0.00 0.095 0.0" rpy="0 0 0"/>
-      <!-- Eje de rotación -->
       <axis xyz="0 1 0"/>
     </joint>
-    <!-- ========================================================= -->
-    <!-- LLANTA DERECHA                                           -->
-    <!-- ========================================================= -->
+    <!-- ================= RIGHT WHEEL ================= -->
     <link name="${prefix}wheel_r_link">
-      <!-- Visual -->
       <visual>
         <origin xyz="0 0 0" rpy="1.5708 0 0"/>
@@ -109,12 +88,10 @@
         </material>
       </visual>
-      <!-- Collision -->
       <collision>
         <origin xyz="0 0 0" rpy="1.5708 0 0"/>
         <geometry>
-          <cylinder radius="0.0325" length="0.02"/>
+          <cylinder radius="0.05" length="0.02"/>
         </geometry>
       </collision>
-      <!-- Inercia -->
       <inertial>
         <mass value="0.2"/>
@@ -125,19 +102,17 @@
       </inertial>
     </link>
-    <!-- Joint rueda derecha -->
+    <!-- Fricción -->
+    <gazebo reference="${prefix}wheel_r_link">
+      <mu1>10.0</mu1>
+      <mu2>10.0</mu2>
+    </gazebo>
     <joint name="${prefix}wheel_r_joint" type="continuous">
       <parent link="${prefix}base_link"/>
       <child link="${prefix}wheel_r_link"/>
-      <!-- Posición lateral derecha -->
       <origin xyz="0.00 -0.095 0.0" rpy="0 0 0"/>
-      <!-- Eje de rotación -->
       <axis xyz="0 1 0"/>
     </joint>
-    <!-- ========================================================= -->
-    <!-- RUEDA CASTER                                              -->
-    <!-- Rueda loca trasera                                       -->
-    <!-- ========================================================= -->
+    <!-- ================= CASTER ================= -->
     <link name="${prefix}caster_link">
-      <!-- Visual -->
       <visual>
         <origin xyz="0 0 0" rpy="0 0 0"/>
@@ -150,5 +125,4 @@
         </material>
       </visual>
-      <!-- Collision -->
       <collision>
         <origin xyz="0 0 0" rpy="0 0 0"/>
@@ -157,5 +131,4 @@
         </geometry>
       </collision>
-      <!-- Inercia -->
       <inertial>
         <mass value="0.05"/>
@@ -166,10 +139,8 @@
       </inertial>
     </link>
-    <!-- Joint caster -->
     <joint name="${prefix}caster_joint" type="fixed">
       <parent link="${prefix}base_link"/>
       <child link="${prefix}caster_link"/>
-      <!-- Posición trasera -->
-      <origin xyz="-0.147 0 -0.0325" rpy="0 0 0"/>
+      <origin xyz="-0.147 0 -0.045" rpy="0 0 0"/>
     </joint>
   </xacro:macro>

File: puzzlebot_ws/src/puzzlebot_ros2/puzzlebot_description/urdf/puzzlebot_control.xacro (robot description, xacro)
@@ -1,17 +1,16 @@
 <?xml version="1.0"?>
 <robot xmlns:xacro="https://www.ros.org/wiki/xacro">
-    <!-- ================= controller ================= -->
     <xacro:macro name="puzzlebot_control" params="prefix">
         <gazebo>
             <plugin filename="gz-sim-sensors-system"
-            name="gz::sim::systems::Sensors">
+                    name="gz::sim::systems::Sensors">
                 <render_engine>ogre2</render_engine>
             </plugin>
             <plugin filename="gz-sim-diff-drive-system"
-            name="gz::sim::systems::DiffDrive">
+                    name="gz::sim::systems::DiffDrive">
                 <left_joint>${prefix}wheel_l_joint</left_joint>
                 <right_joint>${prefix}wheel_r_joint</right_joint>
                 <wheel_separation>0.19</wheel_separation>
-                <wheel_radius>0.0325</wheel_radius>
+                <wheel_radius>0.05</wheel_radius>
                 <topic>${prefix}cmd_vel</topic>
                 <tf_topic>${prefix}diff_drive/tf</tf_topic>
@@ -20,9 +19,9 @@
                 <child_frame_id>${prefix}base_footprint</child_frame_id>
                 <odom_publisher_frequency>50</odom_publisher_frequency>
-                <max_angular_acceleration>1.8</max_angular_acceleration>
-                <max_angular_velocity>13.0</max_angular_velocity>
+                <max_angular_acceleration>1.5</max_angular_acceleration>
+                <max_angular_velocity>8.0</max_angular_velocity>
             </plugin>
             <plugin filename="gz-sim-joint-state-publisher-system"
-            name="gz::sim::systems::JointStatePublisher">
+                    name="gz::sim::systems::JointStatePublisher">
                 <topic>${prefix}joint_states</topic>
                 <update_rate>50</update_rate>
