Commit message: Adjusted robot position again

File: puzzlebot_ws/src/puzzlebot_ros2/puzzlebot_description/urdf/puzzlebot_base.urdf.xacro (robot description, xacro)
@@ -2,4 +2,5 @@
 <robot xmlns:xacro="http://www.ros.org/wiki/xacro">
   <xacro:macro name="puzzlebot_base" params="prefix">
+    <!-- ================= BASE FOOTPRINT ================= -->
     <link name="${prefix}base_footprint"/>
     <!-- ================= BASE LINK ================= -->
@@ -18,12 +19,12 @@
       <!-- Collision -->
       <collision>
-        <origin xyz="-0.052 0 0.05" rpy="0 0 0"/>
+        <origin xyz="0 0 0" rpy="0 0 0"/>
         <geometry>
           <box size="0.20 0.14 0.10"/>
         </geometry>
       </collision>
-      <!-- Inercia corregida -->
+      <!-- Inertial -->
       <inertial>
-        <origin xyz="-0.02 0 -0.02"/>
+        <origin xyz="0 0 0"/>
         <mass value="3.5"/>
         <inertia
@@ -33,9 +34,10 @@
       </inertial>
     </link>
-    <!-- Joint base -->
+    <!-- ================= BASE JOINT ================= -->
     <joint name="${prefix}base_link_joint" type="fixed">
       <parent link="${prefix}base_footprint"/>
       <child link="${prefix}base_link"/>
-      <origin xyz="0.052 0 0.07" rpy="0 0 0"/>
+      <!-- Eleva el robot correctamente -->
+      <origin xyz="0 0 0.05" rpy="0 0 0"/>
     </joint>
     <!-- ================= LEFT WHEEL ================= -->
@@ -73,5 +75,5 @@
       <parent link="${prefix}base_link"/>
       <child link="${prefix}wheel_l_link"/>
-      <origin xyz="0.00 0.095 0.0" rpy="0 0 0"/>
+      <origin xyz="0.00 0.095 0.0025" rpy="0 0 0"/>
       <axis xyz="0 1 0"/>
     </joint>
@@ -110,5 +112,5 @@
       <parent link="${prefix}base_link"/>
       <child link="${prefix}wheel_r_link"/>
-      <origin xyz="0.00 -0.095 0.0" rpy="0 0 0"/>
+      <origin xyz="0.00 -0.095 0.0025" rpy="0 0 0"/>
       <axis xyz="0 1 0"/>
     </joint>
@@ -142,5 +144,5 @@
       <parent link="${prefix}base_link"/>
       <child link="${prefix}caster_link"/>
-      <origin xyz="-0.147 0 -0.045" rpy="0 0 0"/>
+      <origin xyz="-0.147 0 -0.040" rpy="0 0 0"/>
     </joint>
   </xacro:macro>

File: puzzlebot_ws/src/puzzlebot_ros2/puzzlebot_description/urdf/rpi_lidar_sensor.xacro (robot description, xacro)
@@ -29,5 +29,5 @@
     lidar_base_mesh_pos_p:='0.0'
     lidar_base_mesh_pos_w:='0.0'
-    lidar_base_pos_x:='0.0425'
+    lidar_base_pos_x:='0.00'
     lidar_base_pos_y:='0.00'
     lidar_base_pos_z:='0.070'

Commit message: Update robot model files

File: puzzlebot_ws/src/puzzlebot_ros2/puzzlebot_description/urdf/puzzlebot_base.urdf.xacro (robot description, xacro)
@@ -1,19 +1,10 @@
 <?xml version="1.0"?>
 <robot xmlns:xacro="http://www.ros.org/wiki/xacro">
-  <!-- estructura física del Puzzlebot   -->
   <xacro:macro name="puzzlebot_base" params="prefix">
-    <!-- BASE FOOTPRINT                                           -->
-    <!-- Frame base del robot usado para navegación y TF         -->
-    <!-- Normalmente se coloca en el suelo, justo debajo del robot -->
-    <!-- ========================================================= -->
+    <!-- ================= BASE FOOTPRINT ================= -->
     <link name="${prefix}base_footprint"/>
-    <!-- ========================================================= -->
-    <!-- BASE LINK                                                -->
-    <!-- Cuerpo principal del robot                              -->
-    <!-- Contiene mesh visual, colisión e inercia                -->
-    <!-- ========================================================= -->
+    <!-- ================= BASE LINK ================= -->
     <link name="${prefix}base_link">
-      <!-- ================= VISUAL ================= -->
-      <!-- Cómo se ve el robot en RViz/Gazebo -->
+      <!-- Visual -->
       <visual>
         <origin xyz="-0.052 0 0" rpy="0 0 0"/>
@@ -26,37 +17,30 @@
         </material>
       </visual>
-      <!-- ================= COLLISION ================= -->
-      <!-- Geometría usada por Gazebo para física -->
+      <!-- Collision -->
       <collision>
-        <origin xyz="-0.052 0 0.05" rpy="0 0 0"/>
+        <origin xyz="0 0 0" rpy="0 0 0"/>
         <geometry>
           <box size="0.20 0.14 0.10"/>
         </geometry>
       </collision>
-      <!-- ================= INERTIA ================= -->
-      <!-- Propiedades físicas del robot -->
+      <!-- Inertial -->
       <inertial>
         <origin xyz="0 0 0"/>
-        <mass value="2.0"/>
+        <mass value="3.5"/>
         <inertia
-          ixx="0.01" ixy="0.0" ixz="0.0"
-          iyy="0.01" iyz="0.0"
-          izz="0.02"/>
+          ixx="0.06" ixy="0.0" ixz="0.0"
+          iyy="0.08" iyz="0.0"
+          izz="0.10"/>
       </inertial>
     </link>
-    <!-- ========================================================= -->
-    <!-- JOINT BASE FOOTPRINT -> BASE LINK                        -->
-    <!-- Une el frame del suelo con el cuerpo del robot          -->
-    <!-- ========================================================= -->
+    <!-- ================= BASE JOINT ================= -->
     <joint name="${prefix}base_link_joint" type="fixed">
       <parent link="${prefix}base_footprint"/>
       <child link="${prefix}base_link"/>
-      <origin xyz="0.052 0 0.05" rpy="0 0 0"/>
+      <!-- Eleva el robot correctamente -->
+      <origin xyz="0 0 0.05" rpy="0 0 0"/>
     </joint>
-    <!-- ========================================================= -->
-    <!-- LLANTA IZQUIERDA                                         -->
-    <!-- ========================================================= -->
+    <!-- ================= LEFT WHEEL ================= -->
     <link name="${prefix}wheel_l_link">
-      <!-- Visual -->
       <visual>
         <origin xyz="0 0 0" rpy="1.5708 0 0"/>
@@ -69,12 +53,10 @@
         </material>
       </visual>
-      <!-- Collision -->
       <collision>
         <origin xyz="0 0 0" rpy="1.5708 0 0"/>
         <geometry>
-          <cylinder radius="0.0325" length="0.02"/>
+          <cylinder radius="0.05" length="0.02"/>
         </geometry>
       </collision>
-      <!-- Inercia -->
       <inertial>
         <mass value="0.2"/>
@@ -85,18 +67,17 @@
       </inertial>
     </link>
-    <!-- Joint rueda izquierda -->
+    <!-- Fricción -->
+    <gazebo reference="${prefix}wheel_l_link">
+      <mu1>10.0</mu1>
+      <mu2>10.0</mu2>
+    </gazebo>
     <joint name="${prefix}wheel_l_joint" type="continuous">
       <parent link="${prefix}base_link"/>
       <child link="${prefix}wheel_l_link"/>
-      <!-- Posición lateral izquierda -->
-      <origin xyz="0.00 0.095 0.0" rpy="0 0 0"/>
-      <!-- Eje de rotación -->
+      <origin xyz="0.00 0.095 0.0025" rpy="0 0 0"/>
       <axis xyz="0 1 0"/>
     </joint>
-    <!-- ========================================================= -->
-    <!-- LLANTA DERECHA                                           -->
-    <!-- ========================================================= -->
+    <!-- ================= RIGHT WHEEL ================= -->
     <link name="${prefix}wheel_r_link">
-      <!-- Visual -->
       <visual>
         <origin xyz="0 0 0" rpy="1.5708 0 0"/>
@@ -109,12 +90,10 @@
         </material>
       </visual>
-      <!-- Collision -->
       <collision>
         <origin xyz="0 0 0" rpy="1.5708 0 0"/>
         <geometry>
-          <cylinder radius="0.0325" length="0.02"/>
+          <cylinder radius="0.05" length="0.02"/>
         </geometry>
       </collision>
-      <!-- Inercia -->
       <inertial>
         <mass value="0.2"/>
@@ -125,19 +104,17 @@
       </inertial>
     </link>
-    <!-- Joint rueda derecha -->
+    <!-- Fricción -->
+    <gazebo reference="${prefix}wheel_r_link">
+      <mu1>10.0</mu1>
+      <mu2>10.0</mu2>
+    </gazebo>
     <joint name="${prefix}wheel_r_joint" type="continuous">
       <parent link="${prefix}base_link"/>
       <child link="${prefix}wheel_r_link"/>
-      <!-- Posición lateral derecha -->
-      <origin xyz="0.00 -0.095 0.0" rpy="0 0 0"/>
-      <!-- Eje de rotación -->
+      <origin xyz="0.00 -0.095 0.0025" rpy="0 0 0"/>
       <axis xyz="0 1 0"/>
     </joint>
-    <!-- ========================================================= -->
-    <!-- RUEDA CASTER                                              -->
-    <!-- Rueda loca trasera                                       -->
-    <!-- ========================================================= -->
+    <!-- ================= CASTER ================= -->
     <link name="${prefix}caster_link">
-      <!-- Visual -->
       <visual>
         <origin xyz="0 0 0" rpy="0 0 0"/>
@@ -150,5 +127,4 @@
         </material>
       </visual>
-      <!-- Collision -->
       <collision>
         <origin xyz="0 0 0" rpy="0 0 0"/>
@@ -157,5 +133,4 @@
         </geometry>
       </collision>
-      <!-- Inercia -->
       <inertial>
         <mass value="0.05"/>
@@ -166,10 +141,8 @@
       </inertial>
     </link>
-    <!-- Joint caster -->
     <joint name="${prefix}caster_joint" type="fixed">
       <parent link="${prefix}base_link"/>
       <child link="${prefix}caster_link"/>
-      <!-- Posición trasera -->
-      <origin xyz="-0.147 0 -0.045" rpy="0 0 0"/>
+      <origin xyz="-0.147 0 -0.040" rpy="0 0 0"/>
     </joint>
   </xacro:macro>

File: puzzlebot_ws/src/puzzlebot_ros2/puzzlebot_description/urdf/rpi_lidar_sensor.xacro (robot description, xacro)
@@ -29,5 +29,9 @@
     lidar_base_mesh_pos_p:='0.0'
     lidar_base_mesh_pos_w:='0.0'
+<<<<<<< HEAD
     lidar_base_pos_x:='0.0425'
+=======
+    lidar_base_pos_x:='0.00'
+>>>>>>> paul2
     lidar_base_pos_y:='0.00'
     lidar_base_pos_z:='0.070'
@@ -148,3 +152,7 @@
     </gazebo>
     </xacro:macro>
+<<<<<<< HEAD
 </robot>
+=======
+</robot>
+>>>>>>> paul2

Commit message: Adjust nav2 parameters and robot base

File: puzzlebot_ws/src/puzzlebot_ros2/puzzlebot_description/urdf/puzzlebot_base.urdf.xacro (robot description, xacro)
@@ -17,11 +17,11 @@
       <!-- Cómo se ve el robot en RViz/Gazebo -->
       <visual>
-        <origin xyz="-0.052 0 0" rpy="0 0 0"/>
+        <origin xyz="0 0 0" rpy="0 0 0"/>
         <geometry>
           <mesh filename="package://puzzlebot_description/meshes/Puzzlebot_Jetson_Lidar_Edition_Base(1).stl"
                 scale="1 1 1"/>
         </geometry>
-        <material name="white">
-          <color rgba="1.0 1.0 1.0 1.0"/>
+        <material name="red">
+          <color rgba="0.85 0.1 0.1 1.0"/>
         </material>
       </visual>
@@ -29,5 +29,5 @@
       <!-- Geometría usada por Gazebo para física -->
       <collision>
-        <origin xyz="-0.052 0 0.05" rpy="0 0 0"/>
+        <origin xyz="0 0 0" rpy="0 0 0"/>
         <geometry>
           <box size="0.20 0.14 0.10"/>
@@ -45,4 +45,7 @@
       </inertial>
     </link>
+    <gazebo reference="${prefix}base_link">
+      <material>Gazebo/Red</material>
+    </gazebo>
     <!-- ========================================================= -->
     <!-- JOINT BASE FOOTPRINT -> BASE LINK                        -->
@@ -52,5 +55,5 @@
       <parent link="${prefix}base_footprint"/>
       <child link="${prefix}base_link"/>
-      <origin xyz="0.052 0 0.05" rpy="0 0 0"/>
+      <origin xyz="0 0 0.05" rpy="0 0 0"/>
     </joint>
     <!-- ========================================================= -->
@@ -73,5 +76,5 @@
         <origin xyz="0 0 0" rpy="1.5708 0 0"/>
         <geometry>
-          <cylinder radius="0.0325" length="0.02"/>
+          <cylinder radius="0.05" length="0.012"/>
         </geometry>
       </collision>
@@ -90,5 +93,5 @@
       <child link="${prefix}wheel_l_link"/>
       <!-- Posición lateral izquierda -->
-      <origin xyz="0.00 0.095 0.0" rpy="0 0 0"/>
+      <origin xyz="0.052 0.095 -0.0025" rpy="0 0 0"/>
       <!-- Eje de rotación -->
       <axis xyz="0 1 0"/>
@@ -113,5 +116,5 @@
         <origin xyz="0 0 0" rpy="1.5708 0 0"/>
         <geometry>
-          <cylinder radius="0.0325" length="0.02"/>
+          <cylinder radius="0.05" length="0.012"/>
         </geometry>
       </collision>
@@ -130,5 +133,5 @@
       <child link="${prefix}wheel_r_link"/>
       <!-- Posición lateral derecha -->
-      <origin xyz="0.00 -0.095 0.0" rpy="0 0 0"/>
+      <origin xyz="0.052 -0.095 -0.0025" rpy="0 0 0"/>
       <!-- Eje de rotación -->
       <axis xyz="0 1 0"/>
@@ -171,5 +174,5 @@
       <child link="${prefix}caster_link"/>
       <!-- Posición trasera -->
-      <origin xyz="-0.147 0 -0.045" rpy="0 0 0"/>
+      <origin xyz="-0.095 0 -0.03" rpy="0 0 0"/>
     </joint>
   </xacro:macro>

Commit message: Revert "Merge changes into main"
This reverts commit 68031bb93400408ba3ffe1dddb23981f0454d2e2, reversing
changes made to 6c40c0eb5e5ed094ae6d1aead3ea775480c0d6a1.

File: puzzlebot_ws/src/puzzlebot_ros2/puzzlebot_description/urdf/puzzlebot_base.urdf.xacro (robot description, xacro)
@@ -1,31 +1,21 @@
 <?xml version="1.0"?>
 <robot xmlns:xacro="http://www.ros.org/wiki/xacro">
-  <!-- estructura física del Puzzlebot   -->
   <xacro:macro name="puzzlebot_base" params="prefix">
-    <!-- BASE FOOTPRINT                                           -->
-    <!-- Frame base del robot usado para navegación y TF         -->
-    <!-- Normalmente se coloca en el suelo, justo debajo del robot -->
-    <!-- ========================================================= -->
+    <!-- ================= BASE FOOTPRINT ================= -->
     <link name="${prefix}base_footprint"/>
-    <!-- ========================================================= -->
-    <!-- BASE LINK                                                -->
-    <!-- Cuerpo principal del robot                              -->
-    <!-- Contiene mesh visual, colisión e inercia                -->
-    <!-- ========================================================= -->
+    <!-- ================= BASE LINK ================= -->
     <link name="${prefix}base_link">
-      <!-- ================= VISUAL ================= -->
-      <!-- Cómo se ve el robot en RViz/Gazebo -->
+      <!-- Visual -->
       <visual>
-        <origin xyz="0 0 0" rpy="0 0 0"/>
+        <origin xyz="-0.052 0 0" rpy="0 0 0"/>
         <geometry>
           <mesh filename="package://puzzlebot_description/meshes/Puzzlebot_Jetson_Lidar_Edition_Base(1).stl"
                 scale="1 1 1"/>
         </geometry>
-        <material name="red">
-          <color rgba="0.85 0.1 0.1 1.0"/>
+        <material name="white">
+          <color rgba="1.0 1.0 1.0 1.0"/>
         </material>
       </visual>
-      <!-- ================= COLLISION ================= -->
-      <!-- Geometría usada por Gazebo para física -->
+      <!-- Collision -->
       <collision>
         <origin xyz="0 0 0" rpy="0 0 0"/>
@@ -34,32 +24,23 @@
         </geometry>
       </collision>
-      <!-- ================= INERTIA ================= -->
-      <!-- Propiedades físicas del robot -->
+      <!-- Inertial -->
       <inertial>
         <origin xyz="0 0 0"/>
-        <mass value="2.0"/>
+        <mass value="3.5"/>
         <inertia
-          ixx="0.01" ixy="0.0" ixz="0.0"
-          iyy="0.01" iyz="0.0"
-          izz="0.02"/>
+          ixx="0.06" ixy="0.0" ixz="0.0"
+          iyy="0.08" iyz="0.0"
+          izz="0.10"/>
       </inertial>
     </link>
-    <gazebo reference="${prefix}base_link">
-      <material>Gazebo/Red</material>
-    </gazebo>
-    <!-- ========================================================= -->
-    <!-- JOINT BASE FOOTPRINT -> BASE LINK                        -->
-    <!-- Une el frame del suelo con el cuerpo del robot          -->
-    <!-- ========================================================= -->
+    <!-- ================= BASE JOINT ================= -->
     <joint name="${prefix}base_link_joint" type="fixed">
       <parent link="${prefix}base_footprint"/>
       <child link="${prefix}base_link"/>
+      <!-- Eleva el robot correctamente -->
       <origin xyz="0 0 0.05" rpy="0 0 0"/>
     </joint>
-    <!-- ========================================================= -->
-    <!-- LLANTA IZQUIERDA                                         -->
-    <!-- ========================================================= -->
+    <!-- ================= LEFT WHEEL ================= -->
     <link name="${prefix}wheel_l_link">
-      <!-- Visual -->
       <visual>
         <origin xyz="0 0 0" rpy="1.5708 0 0"/>
@@ -72,12 +53,10 @@
         </material>
       </visual>
-      <!-- Collision -->
       <collision>
         <origin xyz="0 0 0" rpy="1.5708 0 0"/>
         <geometry>
-          <cylinder radius="0.05" length="0.012"/>
+          <cylinder radius="0.05" length="0.02"/>
         </geometry>
       </collision>
-      <!-- Inercia -->
       <inertial>
         <mass value="0.2"/>
@@ -88,18 +67,17 @@
       </inertial>
     </link>
-    <!-- Joint rueda izquierda -->
+    <!-- Fricción -->
+    <gazebo reference="${prefix}wheel_l_link">
+      <mu1>10.0</mu1>
+      <mu2>10.0</mu2>
+    </gazebo>
     <joint name="${prefix}wheel_l_joint" type="continuous">
       <parent link="${prefix}base_link"/>
       <child link="${prefix}wheel_l_link"/>
-      <!-- Posición lateral izquierda -->
-      <origin xyz="0.052 0.095 -0.0025" rpy="0 0 0"/>
-      <!-- Eje de rotación -->
+      <origin xyz="0.00 0.095 0.0025" rpy="0 0 0"/>
       <axis xyz="0 1 0"/>
     </joint>
-    <!-- ========================================================= -->
-    <!-- LLANTA DERECHA                                           -->
-    <!-- ========================================================= -->
+    <!-- ================= RIGHT WHEEL ================= -->
     <link name="${prefix}wheel_r_link">
-      <!-- Visual -->
       <visual>
         <origin xyz="0 0 0" rpy="1.5708 0 0"/>
@@ -112,12 +90,10 @@
         </material>
       </visual>
-      <!-- Collision -->
       <collision>
         <origin xyz="0 0 0" rpy="1.5708 0 0"/>
         <geometry>
-          <cylinder radius="0.05" length="0.012"/>
+          <cylinder radius="0.05" length="0.02"/>
         </geometry>
       </collision>
-      <!-- Inercia -->
       <inertial>
         <mass value="0.2"/>
@@ -128,19 +104,17 @@
       </inertial>
     </link>
-    <!-- Joint rueda derecha -->
+    <!-- Fricción -->
+    <gazebo reference="${prefix}wheel_r_link">
+      <mu1>10.0</mu1>
+      <mu2>10.0</mu2>
+    </gazebo>
     <joint name="${prefix}wheel_r_joint" type="continuous">
       <parent link="${prefix}base_link"/>
       <child link="${prefix}wheel_r_link"/>
-      <!-- Posición lateral derecha -->
-      <origin xyz="0.052 -0.095 -0.0025" rpy="0 0 0"/>
-      <!-- Eje de rotación -->
+      <origin xyz="0.00 -0.095 0.0025" rpy="0 0 0"/>
       <axis xyz="0 1 0"/>
     </joint>
-    <!-- ========================================================= -->
-    <!-- RUEDA CASTER                                              -->
-    <!-- Rueda loca trasera                                       -->
-    <!-- ========================================================= -->
+    <!-- ================= CASTER ================= -->
     <link name="${prefix}caster_link">
-      <!-- Visual -->
       <visual>
         <origin xyz="0 0 0" rpy="0 0 0"/>
@@ -153,5 +127,4 @@
         </material>
       </visual>
-      <!-- Collision -->
       <collision>
         <origin xyz="0 0 0" rpy="0 0 0"/>
@@ -160,5 +133,4 @@
         </geometry>
       </collision>
-      <!-- Inercia -->
       <inertial>
         <mass value="0.05"/>
@@ -169,10 +141,8 @@
       </inertial>
     </link>
-    <!-- Joint caster -->
     <joint name="${prefix}caster_joint" type="fixed">
       <parent link="${prefix}base_link"/>
       <child link="${prefix}caster_link"/>
-      <!-- Posición trasera -->
-      <origin xyz="-0.095 0 -0.03" rpy="0 0 0"/>
+      <origin xyz="-0.147 0 -0.040" rpy="0 0 0"/>
     </joint>
   </xacro:macro>

File: puzzlebot_ws/src/puzzlebot_ros2/puzzlebot_description/urdf/rpi_lidar_sensor.xacro (robot description, xacro)
@@ -29,5 +29,9 @@
     lidar_base_mesh_pos_p:='0.0'
     lidar_base_mesh_pos_w:='0.0'
+<<<<<<< HEAD
     lidar_base_pos_x:='0.0425'
+=======
+    lidar_base_pos_x:='0.00'
+>>>>>>> paul2
     lidar_base_pos_y:='0.00'
     lidar_base_pos_z:='0.070'
@@ -148,3 +152,7 @@
     </gazebo>
     </xacro:macro>
+<<<<<<< HEAD
 </robot>
+=======
+</robot>
+>>>>>>> paul2
